File: Skeleton68_underglow/Skeleton68_underglow.kicad_pcb (KiCad board)
At the start: 2 copper layers, 336.6 x 121.7 mm, 170 parts, among them J1 USB_C_Receptacle_USB2.0, SW1 SW_PUSH, SW10 SW_PUSH, SW11 SW_PUSH, SW12 SW_PUSH, SW13 SW_PUSH, SW14 SW_PUSH, SW15 SW_PUSH, SW16 SW_PUSH, SW17 SW_PUSH, SW18 SW_PUSH, SW19 SW_PUSH, SW2 SW_PUSH, SW20 SW_PUSH, SW21 SW_PUSH, SW22 SW_PUSH, SW23 SW_PUSH, SW24 SW_PUSH, SW25 SW_PUSH, SW26 SW_PUSH, SW27 SW_PUSH, SW28 SW_PUSH, SW29 SW_PUSH, SW3 SW_PUSH, SW30 SW_PUSH, SW31 SW_PUSH, SW32 SW_PUSH, SW33 SW_PUSH, SW34 SW_PUSH, SW35 SW_PUSH, SW36 SW_PUSH, SW37 SW_PUSH, SW38 SW_PUSH, SW39 SW_PUSH, SW4 SW_PUSH, SW40 SW_PUSH, SW41 SW_PUSH, SW42 SW_PUSH, SW43 SW_PUSH, SW44 SW_PUSH, SW45 SW_PUSH, SW46 SW_PUSH, SW47 SW_PUSH, SW48 SW_PUSH, SW49 SW_PUSH, SW5 SW_PUSH, SW50 SW_PUSH, SW51 SW_PUSH, SW52 SW_PUSH, SW53 SW_PUSH, SW54 SW_PUSH, SW55 SW_PUSH, SW56 SW_PUSH, SW57 SW_PUSH, SW58 SW_PUSH, SW59 SW_PUSH, SW6 SW_PUSH, SW60 SW_PUSH, SW61 SW_PUSH, SW62 SW_PUSH, SW63 SW_PUSH, SW64 SW_PUSH, SW65 SW_PUSH, SW66 SW_PUSH, SW67 SW_PUSH, SW68 SW_PUSH, SW7 SW_PUSH, SW8 SW_PUSH, SW9 SW_PUSH, U1 ATmega32U4-M, U2 PRTR5V0U2X, Y1 Crystal_GND24

Commit message: routed2
Routing:
- net row2: track 453.9 -> 458.4 mm
- net col14: track 242.0 -> 245.6 mm
- net col9: track 157.6 -> 160.1 mm
- net col12: track 224.4 -> 222.7 mm
- net col1: track 163.9 -> 164.9 mm
- net col4: track 164.3 -> 165.2 mm
- net col3: track 126.7 -> 127.3 mm
- net row1: track 487.9 -> 488.5 mm
- removed copper zone on B.Cu, net GND

Commit message: add underglow version
Parts:
- moved Y1 52.2 mm to (155.8, 60.2), turned to 0 degrees
- moved C2 51.7 mm to (154.7, 55.7)
- moved C1 45.7 mm to (156.8, 55.7)
- moved R4 17.1 mm to (148.2, 79.6), turned to 180 degrees
- moved C3 14.4 mm to (148.2, 77.3), turned to 180 degrees
- moved U1 13.6 mm to (158.4, 72.8)
Routing:
- net GND: track 920.8 -> 870.1 mm, vias 11 -> 8
- net xtal2: track 65.2 -> 15.6 mm, vias 0 -> 2
- net row0: track 433.8 -> 479.7 mm, vias 5 -> 3
- net col13: track 214.8 -> 259.2 mm
- net +5V: track 750.1 -> 792.2 mm
- net xtal1: track 55.7 -> 16.3 mm
- net d+: track 55.0 -> 90.9 mm, vias 0 -> 2
- net led: track 193.8 -> 226.9 mm
- net col10: track 165.9 -> 134.9 mm, vias 0 -> 2
- net row1: track 488.5 -> 458.7 mm, vias 8 -> 7
- net col4: track 165.2 -> 194.5 mm, vias 2 -> 3
- net col1: track 164.9 -> 193.8 mm
- net row3: track 401.6 -> 374.3 mm, vias 7 -> 8
- net col11: track 173.5 -> 152.1 mm
- net Net-(LED3-Pad2): track 67.6 -> 46.3 mm
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- added copper zone on B.Cu, net GND
